File: pcb/hween2017.sch (KiCad schematic (older format))
At the start: 28 parts, among them J1 BATTERY, J2 JTAG, U1 HV509, U2 MSP430FR2100IPW

Commit message: Add new PCB changes and a stencil STL file.
Parts:
- removed D?: D, Diodes_SMD:D_0805, symbol D
- added D12, D13: LED, LEDs:LED_D5.0mm, symbol LED
- added K1, K2: SY-3W-K, halloween:Fujitsu_Relay_SY-3W-K_SPDT_12.5x7.4, symbol SY-3W-K
- added R5: 1 k, Resistors_SMD:R_0805_HandSoldering, symbol R
- R6: renamed from R?; footprint (none) -> Resistors_SMD:R_0805_HandSoldering
- gave numbers to parts that had none: 10
Connections:
- net Earth: now also K1.9 (COIL), K2.5 (COM), K2.6 (COM), K2.9 (COIL)
- net VBAT: now also K1.5 (COM), K1.6 (COM)
- net L_IN: now reaches U2.10 (P2.0)
- net L_IN: now also K1.2 (COIL)
- net L_OUT: now reaches U2.9 (P2.1)
- net L_OUT: now also K2.2 (COIL)
- new net: D12.2 (A), K1.1 (NC)
- new net: D13.2 (A), K1.10 (NO)
- new net: D12.1 (K), D13.1 (K), R5.2
- new net: K2.10 (NO), R5.1
- no-connect marks 16 -> 15

Commit message: Correct the schematic to as-built.
Parts:
- R1, R2, R3: value 44 k -> 20 k
- R6: value 100k -> 1 M
Changed lines of the file:
@@
 P 4500 3550
 F 0 "R3" V 4580 3550 50  0000 C CNN
-F 1 "44 k" V 4500 3550 50  0000 C CNN
+F 1 "20 k" V 4500 3550 50  0000 C CNN
 F 2 "Resistors_SMD:R_0805_HandSoldering" V 4430 3550 50  0001 C CNN
 F 3 "" H 4500 3550 50  0001 C CNN
@@
 P 4500 3350
 F 0 "R2" V 4580 3350 50  0000 C CNN
-F 1 "44 k" V 4500 3350 50  0000 C CNN
+F 1 "20 k" V 4500 3350 50  0000 C CNN
 F 2 "Resistors_SMD:R_0805_HandSoldering" V 4430 3350 50  0001 C CNN
 F 3 "" H 4500 3350 50  0001 C CNN
@@
 P 4500 3150
 F 0 "R1" V 4580 3150 50  0000 C CNN
-F 1 "44 k" V 4500 3150 50  0000 C CNN
+F 1 "20 k" V 4500 3150 50  0000 C CNN
 F 2 "Resistors_SMD:R_0805_HandSoldering" V 4430 3150 50  0001 C CNN
 F 3 "" H 4500 3150 50  0001 C CNN
@@
 P 9850 3000
 F 0 "R6" V 9930 3000 50  0000 C CNN
-F 1 "100k" V 9850 3000 50  0000 C CNN
+F 1 "1 M" V 9850 3000 50  0000 C CNN
 F 2 "Resistors_SMD:R_0805_HandSoldering" V 9780 3000 50  0001 C CNN
 F 3 "" H 9850 3000 50  0001 C CNN

Commit message: Final as-shipped.
Other:
- note added: "<20k series resistor recommended for daylight viewing"
- note added: "Notes"
- note added: "VBAT @ 3.6V nominal"
- note added: "VPP @ 170V"
Changed lines of the file:
@@
 encoding utf-8
 Sheet 1 1
-Title ""
-Date ""
-Rev ""
+Title "Nixie Halloween Prop"
+Date "2017-10-19"
+Rev "RC2"
 Comp ""
 Comment1 ""
@@
 Text GLabel 2650 6000 1    60   Input ~ 0
 L_IN
+Text Notes 6400 7000 0    60   ~ 0
+VBAT @ 3.6V nominal
+Text Notes 6400 7100 0    60   ~ 0
+VPP @ 170V
+Text Notes 6300 6900 0    60   ~ 12
+Notes
+Text Notes 6400 7200 0    60   ~ 0
+<20k series resistor recommended for daylight viewing
 $EndSCHEMATC
